File: UniversalPowerModule/UPM_pcb_v1-0.sch (EAGLE design)
At the start: 27 parts, among them Q1 DMP4047SK3, U1 TLV1117_4TERM-33_DCY, U2 TLV1117_4TERM-50_DCY

Commit message: UPM+CAN v1 sent to FAB
Parts:
- removed D2: VISHAY_SMA6F, npol-discrete:VISHAY_SMA6F
- removed TP1, TP3: (no value), microbuilder:TESTPOINT0.1"
- added C4, C5, C6: 0.1uF, rcl:C-USC0603
- added C7, C8: 22nF, rcl:C-USC0603
- added C9: 10nF, rcl:C-USC0603
- added D3: (no value), SparkFun-DiscreteSemi:DIODE1N4148
- added JP6: M02POLAR_LOCK, SparkFun-Connectors:M02POLAR_LOCK
- added JP7: M10X2, SparkFun-Connectors:M10X2
- added LED4: green, SparkFun-LED:LED0603
- added LED5: blue, SparkFun-LED:LED0603
- added Q2: INFINEON_2N7002_DW, npol-discrete:INFINEON_2N7002_DW
- added R5: 120, rcl:R-US_R0603
- added R6, R7: 10k, rcl:R-US_R0603
- added R8, R9: 330, rcl:R-US_R0603
- added TP6, TP7, TP8: (no value), microbuilder:TESTPOINT0.1"
- added U3: MCP2515-SO, npol-digital:MCP2515-SO
- added U4: MCP2562-SN, npol-digital:MCP2562-SN
- added Y1: 8MHz, SparkFun-FreqCtrl:CRYSTALHC49UV
- C3: value 100uF -> 1000uF; device rcl:CPOL-USE2.5-5 -> rcl:CPOL-USE5-13
- JP1: value M022.54MM_SCREWTERM -> (none); device SparkFun-Connectors:M022.54MM_SCREWTERM -> SparkFun-Connectors:M04LOCK
- JP2: value M02POLAR_LOCK -> ONSHORE_OSTYK21102030; device SparkFun-Connectors:M02POLAR_LOCK -> npol-connectors:ONSHORE_OSTYK21102030
Connections:
- removed net +3.3V: C1.+, JP5.2, R4.2, TP4.P$1, U1.OUT, U1.TAB
- new net +3V3: C1.+, C4.1, C5.1, D3.C, JP5.2, JP7.13, JP7.14, R4.2, R7.2, R8.1, R9.1, TP4.P$1, U1.OUT, U1.TAB, U3.VDD, U4.VIO
- new net /CS: JP1.4, JP7.4, U3./CS
- new net /INT: JP7.5, U3./INT
- new net /RESET: JP7.2, R6.2, U3./RESET
- new net /RX0BF: JP7.8, U3./RX0BF
- new net /RX1BF: JP7.7, U3./RX1BF
- new net /TX0RTS: JP7.12, U3./TX0RTS
- new net /TX1RTS: JP7.9, U3./TX1RTS
- new net /TX2RTS: JP7.10, U3./TX2RTS
- new net CANH: JP6.2, R5.2, TP7.P$1, U4.CANH
- new net CANL: JP6.1, R5.1, TP8.P$1, U4.CANL
- new net CLKOUT: TP6.P$1, U3.CLKOUT/SOF
- new net MISO: JP1.3, JP7.6, U3.SO
- new net MOSI: JP1.2, JP7.3, U3.SI
- new net N$10: LED4.A, R8.2
- new net N$11: LED5.A, R9.2
- new net N$7: C9.1, D3.A, R6.1, R7.1
- new net N$8: LED5.C, Q2G$2.DRAIN
- new net RXCAN: Q2G$2.GATE, U3.RXCAN, U4.RXD
- new net SCK: JP1.1, JP7.1, U3.SCK
- new net STBY: JP7.11, U4.STBY
- new net TXCAN: Q2G$1.GATE, U3.TXCAN, U4.TXD
- new net XTAL1: C8.1, U3.OSC1, Y1.2
- new net XTAL2: C7.1, U3.OSC2, Y1.1
- net +12V: now also JP7.15, JP7.16
- net +5V: now also C6.1, JP7.17, JP7.18, U4.VDD
- net GND: now also C4.2, C5.2, C6.2, C7.2, C8.2, C9.2, D1.A, JP7.19, JP7.20, Q2G$1.SOURCE, Q2G$2.SOURCE, U3.VSS, U4.VSS; no longer D2.K, TP3.P$1
- net N$1: now also LED4.C, Q2G$1.DRAIN; no longer D1.A, D2.A
- net VIN+: now also JP2.P2; no longer JP1.1, JP2.1, TP1.P$1
- net VIN-: now also JP2.P1; no longer JP1.2, JP2.2
Other:
- note added: "CAN Indicator LEDS"
- note added: "CAN Section"
- note added: "Header"
- note added: "Power Section"
- note added: "TXD,STBY have internal pullup"
- note added: "TXnRTS have internal pullup"
- note added: "Team NSH Project CLEANUP Robotics Capstone 16-474"
- note removed: "TODO: Diode for LDOs LEDs for all rails header for parent"
- note removed: "Team CLEANUP Robotics Capstone 16-474"
