File: MobilityEliminationController/MobilityEliminationController.sch (EAGLE design)
At the start: 93 parts, among them Q1 INFINEON_2N7002_DW, Q2 INFINEON_2N7002_DW, Q3 INFINEON_2N7002_DW, Q4 INFINEON_2N7002_DW, U1 MSP430F5521/5/7/9_PN80

Commit message: Mostly done, but brd file is blank
Parts:
- removed C13: 0.1uF, rcl:C-USC0603
- removed C14: 1nF, rcl:C-USC0603
- removed D1, D2, D3, D4, D5, D6: 1N5400, diode:1N5400
- removed JP12: M02LOCK, SparkFun-Connectors:M02LOCK
- removed R19, R25: 1k, rcl:R-US_R0603
- removed RLY1, RLY2, RLY3, RLY4, RLY5, U$6: TE_V23201-C1001-A502, npol-electromechanical:TE_V23201-C1001-A502
- removed U$10: ONSHORE_OSTYK21102030, npol-connectors:ONSHORE_OSTYK21102030
- removed U$9: ACS712, npol:ACS712
- added H1, H2, H3, H4: MOUNT-PAD-ROUND3.2, holes:MOUNT-PAD-ROUND3.2
- added JP15: (no value), SparkFun-Connectors:M04SCREW
- added JP16: (no value), SparkFun-Connectors:M03X22X3_SILK_SM
- added LED10, LED11: Status: Red, SparkFun-LED:LED0603
- added Q5, Q6: INFINEON_2N7002_DW, npol-discrete:INFINEON_2N7002_DW
- added R28, R29: 100k, rcl:R-US_R0603
- added R30, R31, R32, R33: 10k, rcl:R-US_R0603
- added R34: 330, rcl:R-US_R0603
- added R35: 1k, rcl:R-US_R0603
- added TP2, TP3: (no value), microbuilder:TESTPOINT0.1"
- JP10: value (none) -> M02LOCK; device SparkFun-Connectors:M03SCREW -> SparkFun-Connectors:M02LOCK
- JP7: value ONSHORE_OSTYK21102030 -> (none); device npol-connectors:ONSHORE_OSTYK21102030 -> SparkFun-Connectors:M04SCREW
- JP8: value ONSHORE_OSTYK21102030 -> M023.5MM; device npol-connectors:ONSHORE_OSTYK21102030 -> SparkFun-Connectors:M023.5MM
- JP9: device SparkFun-Connectors:M03SCREW -> SparkFun-Connectors:M07
- Q3, Q4: value INFINEON_2N7002_DW -> BS250F; device npol-discrete:INFINEON_2N7002_DW -> SparkFun-DiscreteSemi:MOSFET-PCHANNELSMD
- R22: value 10k -> 330
- R23: value 10k -> 100k
- SJ1, SJ2, SJ3, SJ4: device microbuilder:SOLDERJUMPER_2WAY -> microbuilder:SOLDERJUMPER_2WAY0603
- renumbered LED6 to LED12, LED7 to LED13, U$7 to U3, U$8 to U2
Connections:
- net DBG_LED renamed DBG_LED1
- net N$18 renamed RELAY3_CNTRL
- net N$19 renamed RELAY4_CNTRL
- net N$32 renamed RELAY3_LED_A
- removed net DRILL_GND: D2.A, D4.A, JP8.P2, RLY2.5.1, RLY2.5.2, RLY4.5.1, RLY4.5.2
- removed net DRILL_ISENSE: R22.1, R23.2
- removed net DRILL_PWR: D5.C, JP8.P1, U$6.4.1, U$6.4.2
- removed net N$15: Q2G$2.DRAIN, RLY4.2
- removed net N$16: Q1G$1.GATE, R18.2, U31.Y
- removed net N$17: Q1G$2.GATE, R19.2, U32.Y
- removed net N$21: JP7.P1, U$9.IP-@1, U$9.IP-@2
- removed net N$24: D1.A, D2.C, RLY1.5.1, RLY1.5.2, RLY2.4.1, RLY2.4.2, U$9.IP+@1, U$9.IP+@2
- removed net N$30: LED12.A, R18.1
- removed net N$31: LED13.A, R19.1
- removed net N$34: D6.A, JP10.2, RLY5.5.1, RLY5.5.2
- removed net N$35: C14.1, U$9.FLTR
- removed net N$37: OK1.BAS, R25.2
- removed net N$39: JP12.1, R25.1
- removed net STEPPER_PWR: D6.C, RLY5.4.1, RLY5.4.2, U$10.P1
- new net 12VSENSE: R29.1, R30.2, U1.P5.1/A9/VREF-
- new net 5VSENSE: R23.1, R28.2, U1.P5.0/A8/VREF+
- new net DBG_LED2: R22.2, TP2.P$1, U1.P2.2/TA2CLK/SMCLK
- new net DBG_LED3: R34.2, TP3.P$1, U1.P7.7/TB0CLK/MCLK
- new net DRILL_ISENSE_/FAULT: JP9.5, U1.P1.3/TA0.2
- new net DRILL_ISENSE_FAULT_EN: JP9.6, U1.P6.0/CB0/A0
- new net DRILL_ISENSE_VIOUT: JP9.3, U1.P6.2/CB2/A2
- new net DRILL_ISENSE_VZCR: JP9.4, U1.P6.1/CB1/A1
- new net DRILL_RELAY_1: JP7.4, Q1G$1.DRAIN
- new net DRILL_RELAY_2: JP7.3, Q1G$2.DRAIN
- new net DRILL_RELAY_3: JP7.2, Q2G$1.DRAIN
- new net DRILL_RELAY_4: JP7.1, Q2G$2.DRAIN
- new net ESTOP_RELAY: JP8.2, Q5G$1.SOURCE, Q5G$2.SOURCE
- new net NU_P6.3: JP16.5, U1.P6.3/CB3/A3
- new net NU_P6.4: JP16.6, U1.P6.4/CB4/A4
- new net NU_P6.5: JP16.3, U1.P6.5/CB5/A5
- new net NU_P6.6: JP16.4, U1.P6.6/CB6/A6
- new net NU_P6.7: JP16.1, U1.P6.7/CB7/A7
- new net NU_P7.0: U1.P7.0/CB8/A12
- new net RC_PWR: JP10.1, JP6.2
- new net RELAY1_CNTRL: Q1G$1.GATE, R35.2, U31.Y
- new net RELAY1_LED_A: LED12.A, R35.1
- new net RELAY2_CNTRL: Q1G$2.GATE, R18.2, U32.Y
- new net VOC: JP9.7
- new net VTAP_EN: Q4.G, Q6G$2.DRAIN, R32.1
- net +12V: now also JP8.1, Q4.S, R32.2; no longer RLY1.1, RLY2.1, RLY3.1, RLY4.1, RLY5.1, U$6.1
- net +3V3: now also JP9.2, LED1.A, R33.2; no longer R5.2
- net +5V: now also JP10.2, JP15.4, Q3.S, R31.2; no longer C13.1, JP6.2, JP9.3, U$9.VCC
- net CAN_/CS: now also U1.P2.3/TA2.0
- net CAN_/INT: now also U1.P2.4/TA2.1
- net CAN_/RX0BF: now also U1.P2.5/TA2.2
- net CAN_/RX1BF: now also U1.P2.6/RTCCLK/DMAE0
- net CAN_STBY: now also U1.P2.7/UCB0STE/UCA0CLK
- net DRILL_EN: now also U1.P7.6/TB0.4
- net DRILL_S1: now also U1.P7.5/TB0.3
- net DRILL_S2: now also U1.P7.4/TB0.2
- net ESTOP_LOCAL: now also Q5G$1.GATE, Q5G$2.GATE, U1.P1.4/TA0.3; no longer Q3G$1.GATE, Q4G$1.GATE
- net GND: now also H1.MOUNT, H2.MOUNT, H3.MOUNT, H4.MOUNT, JP16.2, JP9.1, LED10.C, LED11.C, Q5G$1.DRAIN, Q5G$2.DRAIN, Q6G$1.SOURCE, Q6G$2.SOURCE, R28.1, R30.1, R5.1; no longer C13.2, C14.2, JP10.1, JP12.2, LED1.C, Q3G$1.SOURCE, Q4G$1.SOURCE, R23.1, U$10.P2, U$9.GND
- net LOWER_SWITCH: now also U1.P2.0/TA1.1
- net N$10: now also Q3.G, Q6G$1.DRAIN, R31.1; no longer D3.A, D4.C, JP7.P2, RLY3.5.1, RLY3.5.2, RLY4.4.1, RLY4.4.2
- net N$11: now also Q4.D, R29.2; no longer Q1G$1.DRAIN, RLY1.2
- net N$12: now also Q6G$1.GATE, Q6G$2.GATE, R33.1; no longer D1.C, D3.C, D5.A, RLY1.4.1, RLY1.4.2, RLY3.4.1, RLY3.4.2, U$6.5.1, U$6.5.2
- net N$13: now also OK1.COL; no longer Q1G$2.DRAIN, RLY2.2
- net N$14: now also LED13.A, R18.1; no longer Q2G$1.DRAIN, RLY3.2
- net N$2: now also LED1.C, R5.2; no longer LED1.A, R5.1
- net N$36: now also LED11.A, R34.1; no longer Q4G$1.DRAIN, RLY5.2
- net N$8: now also LED10.A, R22.1; no longer R22.2, U$9.VOUT
- net N$9: now also Q3.D, R23.2; no longer Q3G$1.DRAIN, U$6.2
- net STAT_ERR: now also U1.P4.7/PM_NONE
- net STAT_OK: now also U1.P5.7/TB0.1
- net STAT_WARN: now also U1.P5.6/TB0.0
- net STEPPER_DIR: now also JP15.2, U1.P7.1/CB9/A13; no longer JP9.1
- net STEPPER_EN: now also JP15.3, U1.P7.2/CB10/A14; no longer JP9.2
- net STEPPER_STEP: now also JP15.1, U1.P1.2/TA0.1; no longer JP10.3
- net UPPER_SWITCH: now also U1.P2.1/TA1.2
Other:
- note added: "ACS709 Current Sensor"
- note added: "ESTOP Relay Output shared with Drill and Stepper ESTOP relays"
- note added: "VOC Unused"
- note removed: "ESTOP Test"
- note removed: "TODO: Hookup to pins"
- moved on the sheet: JP8, LED1, LED5, R18, R5, R9, TP1
