File: MobilityEliminationController/MobilityEliminationController.sch (EAGLE design)
At the start: 94 parts, among them Q1 INFINEON_2N7002_DW, Q2 INFINEON_2N7002_DW, Q3 BS250F, Q4 BS250F, Q5 INFINEON_2N7002_DW, Q6 INFINEON_2N7002_DW, U1 MSP430F5521/5/7/9_PN80, U2 SN74LV74, U3 SN74LV08

Commit message: Mob/Elim controller ready for fab
Parts:
- removed JP16: (no value), SparkFun-Connectors:M03X22X3_SILK_SM
- removed LED12, LED13: (no value), SparkFun-LED:LED0603
- removed OK1: 4N35, optocoupler:4N35
- removed R35: 1k, rcl:R-US_R0603
- added J11: M10X2, SparkFun-Connectors:M10X2
- added JP12: M02LOCK, SparkFun-Connectors:M02LOCK
- added LED6: Status: Yellow, SparkFun-LED:LED0603
- added LED7: Status: Red, SparkFun-LED:LED0603
- added Q7: INFINEON_2N7002_DW, npol-discrete:INFINEON_2N7002_DW
- added R19: 100k, rcl:R-US_R0603
- added R25: 620, rcl:R-US_R0603
- added U4: SN74LV08, npol-digital:SN74LV08
- C1: value 1nF -> 10uF; device rcl:C-USC0603 -> rcl:C-USC0805
- C10: value 0.1uF -> 1nF
- C2, C3: value 1nF -> 0.1uF
- C4: value 220nF -> 470nF
- C5: value 220nF -> 0.1uF
- C6, C7: value 0.1uF -> 220nF
- C8: value 470nF -> 1nF
- C9: value 10uF -> 1nF; device rcl:C-USC0805 -> rcl:C-USC0603
- JP1: value M10X2 -> (none); device SparkFun-Connectors:M10X2 -> SparkFun-Connectors:M03X22X3_SILK_SM
- JP10: value M02LOCK -> M023.5MM; device SparkFun-Connectors:M02LOCK -> SparkFun-Connectors:M023.5MM
- JP14: value M023.5MM -> (none); device SparkFun-Connectors:M023.5MM -> SparkFun-Connectors:M04SCREW
- JP15: device SparkFun-Connectors:M04SCREW -> SparkFun-Connectors:M07
- JP2: value (none) -> M02LOCK; device SparkFun-Connectors:M03LOCK -> SparkFun-Connectors:M02LOCK
- JP5: value M02LOCK -> (none); device SparkFun-Connectors:M02LOCK -> SparkFun-Connectors:M03LOCK
- JP8: value M023.5MM -> M02LOCK; device SparkFun-Connectors:M023.5MM -> SparkFun-Connectors:M02LOCK
- JP9: value (none) -> M02POLAR_LOCK; device SparkFun-Connectors:M07 -> SparkFun-Connectors:M02POLAR_LOCK
- LED1: value 3V3 OK -> Status: Red
- LED10, LED11: value Status: Red -> (none)
- LED2: value Status: Green -> Status: Red
- LED3: value Status: Yellow -> Status: Red
- LED4: value Status: Red -> 3V3 OK
- LED5: value Status: Red -> Status: Green
- R1: value 47k -> 330
- R10, R11, R3: value 10k -> 330
- R12, R2: value 0 -> 330
- R13: value 1M -> 0
- R14, R15, R16, R17: value 0 -> 10k
- R18, R21: value 1k -> 100k
- R20: value 1k -> 10k
- R22, R7, R9: value 330 -> 10k
- R23: value 100k -> 10k
- R24: value 620 -> 10k
- R27, R33, R4: value 10k -> 0
- R28: value 100k -> 0
- R29: value 100k -> 1k
- R30, R31, R32: value 10k -> 1k
- R34: value 330 -> 0
- R5: value 330 -> 1M
- R6: value 330 -> 47k
- U2: value SN74LV74 -> LTV-817; device npol-digital:SN74LV74 -> npol-digital:LTV-817
- U3: value SN74LV08 -> SN74LV74; device npol-digital:SN74LV08 -> npol-digital:SN74LV74
Connections:
- removed net N$38: OK1.A, R24.1
- new net ESTOP_LOCAL_INV: Q5G$1.GATE, U2.4
- net +12V: now also J11.15, J11.16, JP13.1, R20.2; no longer JP1.15, JP1.16, JP8.1, R32.2
- net +3V3: now also C1.1, C2.1, C3.1, J11.13, J11.14, JP15.2, JP2.1, JP5.2, LED4.A, R23.2, R24.2, R26.1, R28.1, R34.1, R4.2, R6.2, U41.VCC; no longer C6.1, C7.1, C9.1, JP1.13, JP1.14, JP2.2, JP5.1, JP9.2, LED1.A, R1.2, R14.2, R15.1, R17.1, R2.2, R26.2, U21.VCC
- net +5V: now also J11.17, J11.18, JP7.4, JP8.2, R17.2; no longer JP1.17, JP1.18, JP10.2, JP15.4, R31.2
- net 12VSENSE: now also R21.1, R22.2; no longer R29.1, R30.2
- net 5VSENSE: now also R18.1, R19.2; no longer R23.1, R28.2
- net AVCC: now also C5.1, R4.1; no longer C10.1, R2.1
- net CAN_/CS: now also J11.4; no longer JP1.4
- net CAN_/INT: now also J11.5; no longer JP1.5
- net CAN_/RESET: now also J11.2; no longer JP1.2
- net CAN_/RX0BF: now also J11.8; no longer JP1.8
- net CAN_/RX1BF: now also J11.7; no longer JP1.7
- net CAN_/TX0RTS: now also J11.12; no longer JP1.12
- net CAN_/TX1RTS: now also J11.9; no longer JP1.9
- net CAN_/TX2RTS: now also J11.10; no longer JP1.10
- net CAN_MISO: now also J11.6; no longer JP1.6
- net CAN_MOSI: now also J11.3; no longer JP1.3
- net CAN_SCK: now also J11.1; no longer JP1.1
- net CAN_STBY: now also J11.11; no longer JP1.11
- net DBG_LED1: now also R1.2; no longer R9.2
- net DBG_LED2: now also R2.2; no longer R22.2
- net DBG_LED3: now also R3.2; no longer R34.2
- net DBG_RXD: now also R7.2; no longer R3.2
- net DBG_TXD: now also R9.2; no longer R4.2
- net DRILL_EN: now also U31.CLK, U32.CLK, U41.B, U42.A, U43.B, U44.A; no longer U21.CLK, U22.CLK, U31.B, U32.A, U33.B, U34.A
- net DRILL_ISENSE_/FAULT: now also JP15.5; no longer JP9.5
- net DRILL_ISENSE_FAULT_EN: now also JP15.6; no longer JP9.6
- net DRILL_ISENSE_VIOUT: now also JP15.3; no longer JP9.3
- net DRILL_ISENSE_VZCR: now also JP15.4; no longer JP9.4
- net DRILL_RELAY_1: now also JP14.4, Q6G$1.DRAIN; no longer JP7.4, Q1G$1.DRAIN
- net DRILL_RELAY_2: now also JP14.3, Q6G$2.DRAIN; no longer JP7.3, Q1G$2.DRAIN
- net DRILL_RELAY_3: now also JP14.2, Q7G$1.DRAIN; no longer JP7.2, Q2G$1.DRAIN
- net DRILL_RELAY_4: now also JP14.1, Q7G$2.DRAIN; no longer JP7.1, Q2G$2.DRAIN
- net DRILL_S1: now also U31.D; no longer U21.D
- net DRILL_S2: now also U32.D; no longer U22.D
- net ESTOP+: now also JP9.1, R25.2; no longer JP11.2, R24.2
- net ESTOP-: now also JP9.2, U2.2; no longer JP11.1, OK1.C
- net ESTOP_LOCAL: now also JP12.1, Q1G$1.GATE, Q1G$2.GATE, Q5G$1.DRAIN, R13.1, R26.2; no longer Q5G$1.GATE, Q5G$2.GATE, R12.1
- net ESTOP_RELAY: now also JP13.2, Q1G$1.SOURCE, Q1G$2.SOURCE; no longer JP8.2, Q5G$1.SOURCE, Q5G$2.SOURCE
- net GND: now also J11.19, J11.20, JP1.2, JP10.1, JP11.1, JP12.2, JP15.1, LED1.C, LED6.C, LED7.C, Q1G$1.DRAIN, Q1G$2.DRAIN, Q5G$1.SOURCE, Q7G$1.SOURCE, Q7G$2.SOURCE, R14.1, R15.1, R19.1, R22.1, R7.1, R8.1, R9.1, U2.3, U41.GND; no longer JP1.19, JP1.20, JP13.1, JP14.1, JP16.2, JP9.1, LED12.C, LED13.C, LED4.C, OK1.EMI, Q1G$1.SOURCE, Q1G$2.SOURCE, Q5G$1.DRAIN, Q5G$2.DRAIN, R10.1, R11.1, R13.1, R28.1, R3.1, R30.1, R4.1, U21.GND
- net LOWER_SWITCH: now also JP11.2, R24.1; no longer JP14.2, R27.1
- net N$1: now also JP2.2; no longer JP5.2
- net N$10: now also Q2G$1.DRAIN, R17.1; no longer Q6G$1.DRAIN, R31.1
- net N$11: now also R21.2; no longer R29.2
- net N$12: now also Q2G$1.GATE, Q2G$2.GATE, R16.1; no longer Q6G$1.GATE, Q6G$2.GATE, R33.1
- net N$13: now also R25.1, U2.1; no longer OK1.COL
- net N$14: now also LED9.A, R30.1; no longer LED13.A, R18.1
- net N$2: now also LED4.C, R8.2; no longer LED1.C, R5.2
- net N$20: now also U31.Q, U41.A; no longer U21.Q, U31.A
- net N$22: now also U31./Q, U42.B; no longer U21./Q, U32.B
- net N$23: now also U32.Q, U43.A; no longer U22.Q, U33.A
- net N$25: now also U32./Q, U44.B; no longer U22./Q, U34.B
- net N$26: now also R27.1, U31./PRE; no longer R14.1, U21./PRE
- net N$27: now also R28.2, U31./CLR; no longer R15.2, U21./CLR
- net N$28: now also R33.1, U32./PRE; no longer R16.1, U22./PRE
- net N$29: now also R34.2, U32./CLR; no longer R17.2, U22./CLR
- net N$3: now also LED5.A, R10.1; no longer LED2.A, R6.1
- net N$33: now also LED11.A, R32.1; no longer LED9.A, R21.1
- net N$36: now also LED3.A, R3.1; no longer LED11.A, R34.1
- net N$4: now also LED6.A, R11.1; no longer LED3.A, R7.1
- net N$5: now also LED7.A, R12.1; no longer LED4.A, R8.1
- net N$6: now also LED1.A, R1.1; no longer LED5.A, R9.1
- net N$7: now also R5.2; no longer R13.2
- net N$8: now also LED2.A, R2.1; no longer LED10.A, R22.1
- net N$9: now also R18.2; no longer R23.2
- net NU_P6.3: now also JP1.5; no longer JP16.5
- net NU_P6.4: now also JP1.6; no longer JP16.6
- net NU_P6.5: now also JP1.3; no longer JP16.3
- net NU_P6.6: now also JP1.4; no longer JP16.4
- net NU_P6.7: now also JP1.1; no longer JP16.1
- net RC_PWR: now also JP8.1; no longer JP10.1
- net RC_RXD: now also R14.2; no longer R10.2
- net RC_S3: now also R13.2; no longer R12.2
- net RC_TXD: now also R15.2; no longer R11.2
- net RELAY1_CNTRL: now also Q6G$1.GATE, R29.2, U41.Y; no longer Q1G$1.GATE, R35.2, U31.Y
- net RELAY1_LED_A: now also LED8.A, R29.1; no longer LED12.A, R35.1
- net RELAY2_CNTRL: now also Q6G$2.GATE, R30.2, U42.Y; no longer Q1G$2.GATE, R18.2, U32.Y
- net RELAY3_CNTRL: now also Q7G$1.GATE, R31.2, U43.Y; no longer Q2G$1.GATE, R20.2, U33.Y
- net RELAY3_LED_A: now also LED10.A, R31.1; no longer LED8.A, R20.1
- net RELAY4_CNTRL: now also Q7G$2.GATE, R32.2, U44.Y; no longer Q2G$2.GATE, R21.2, U34.Y
- net SBWTDIO: now also C8.1, R6.1; no longer C1.1, R1.1
- net STAT_ERR: now also R12.2; no longer R8.2
- net STAT_OK: now also R10.2; no longer R6.2
- net STAT_WARN: now also R11.2; no longer R7.2
- net STEPPER_DIR: now also JP7.2; no longer JP15.2
- net STEPPER_EN: now also JP7.3; no longer JP15.3
- net STEPPER_STEP: now also JP7.1; no longer JP15.1
- net UPPER_SWITCH: now also JP10.2, R23.1; no longer JP13.2, R26.1
- net V18: now also C7.1; no longer C5.1
- net VCC_TARGET: now also JP5.1; no longer JP2.1
- net VCC_TOOL: now also JP5.3; no longer JP2.3
- net VCORE: now also C4.1; no longer C8.1
- net VOC: now also JP15.7; no longer JP9.7
- net VTAP_EN: now also Q2G$2.DRAIN, R20.1; no longer Q6G$2.DRAIN, R32.1
- net VUSB: now also C6.1; no longer C4.1
- net XT2IN: now also C9.1; no longer C2.1
- net XT2OUT: now also C10.1; no longer C3.1

Commit message: Power Controller, Elim-Mobility Controller, and PC2CAN sent to FAB
Parts:
- added LED12: (no value), SparkFun-LED:LED0603
- added R35: 10k, rcl:R-US_R0603
- added R36: 330, rcl:R-US_R0603
- added R37: 10M, rcl:R-US_R0603
Connections:
- new net N$15: Q5G$2.DRAIN, R36.2
- new net N$16: LED12.C, R36.1
- net +3V3: now also LED12.A, R35.1
- net ESTOP_LOCAL: now also Q5G$2.GATE
- net ESTOP_LOCAL_INV: now also R35.2, R37.1
- net GND: now also Q5G$2.SOURCE, R37.2
