File: PC2CAN/PC2CAN.brd (EAGLE design)
At the start: 57.1 x 63.5 mm, 97 parts, among them J11 M10X2, Q1 INFINEON_2N7002_DW, Q2 INFINEON_2N7002_DW, Q3 BS250F, Q4 BS250F, Q5 INFINEON_2N7002_DW, Q6 INFINEON_2N7002_DW, Q7 INFINEON_2N7002_DW, U1 MSP430F5521/5/7/9_PN80, U2 LTV-817, U3 SN74LV74, U4 SN74LV08

Commit message: Removed irrelevant circuits for PC2CAN and Power Controller
Parts:
- removed C11, C12: 0.1uF, rcl:C0603
- removed JP10, JP11, JP13: M023.5MM, SparkFun-Connectors:SCREWTERMINAL-3.5MM-2
- removed JP14, JP7: (no value), SparkFun-Connectors:SCREWTERMINAL-3.5MM-4
- removed JP15: (no value), SparkFun-Connectors:1X07
- removed JP6: (no value), SparkFun-Connectors:1X05_LOCK
- removed JP8: M02LOCK, SparkFun-Connectors:1X02_LOCK
- removed LED10, LED11, LED8, LED9: (no value), SparkFun-LED:LED-0603
- removed Q1, Q6, Q7: INFINEON_2N7002_DW, npol-discrete:INFINEON_SOT363
- removed R13, R27, R28, R33, R34: 0, rcl:R0603
- removed R23, R24: 10k, rcl:R0603
- removed R29, R30, R31, R32: 1k, rcl:R0603
- removed U3: SN74LV74, npol-digital:TI_D_R-PDSO-G14_SOIC14
- removed U4: SN74LV08, npol-digital:TI_D_R-PDSO-G14_SOIC14
Connections:
- removed net DRILL_RELAY_1: JP14.4, Q6.6
- removed net DRILL_RELAY_2: JP14.3, Q6.3
- removed net DRILL_RELAY_3: JP14.2, Q7.6
- removed net DRILL_RELAY_4: JP14.1, Q7.3
- removed net ESTOP_RELAY: JP13.2, Q1.1, Q1.4
- removed net N$14: LED9.A, R30.1
- removed net N$20: U3.5, U4.1
- removed net N$22: U3.6, U4.5
- removed net N$23: U3.9, U4.9
- removed net N$25: U3.8, U4.13
- removed net N$26: R27.1, U3.4
- removed net N$27: R28.2, U3.1
- removed net N$28: R33.1, U3.10
- removed net N$29: R34.2, U3.13
- removed net N$33: LED11.A, R32.1
- removed net RC_PWR: JP6.2, JP8.1
- removed net RC_S3: JP6.5, R13.2
- removed net RELAY1_CNTRL: Q6.2, R29.2, U4.3
- removed net RELAY1_LED_A: LED8.A, R29.1
- removed net RELAY2_CNTRL: Q6.5, R30.2, U4.6
- removed net RELAY3_CNTRL: Q7.2, R31.2, U4.8
- removed net RELAY3_LED_A: LED10.A, R31.1
- removed net RELAY4_CNTRL: Q7.5, R32.2, U4.11
- removed net VOC: JP15.7
- net +12V: no longer JP13.1
- net +3V3: no longer C11.1, C12.1, JP15.2, R23.2, R24.2, R27.2, R28.1, R33.2, R34.1, U3.14, U4.14
- net +5V: no longer JP7.4, JP8.2
- net DRILL_EN: no longer U3.11, U3.3, U4.10, U4.12, U4.2, U4.4
- net DRILL_ISENSE_/FAULT: no longer JP15.5
- net DRILL_ISENSE_FAULT_EN: no longer JP15.6
- net DRILL_ISENSE_VIOUT: no longer JP15.3
- net DRILL_ISENSE_VZCR: no longer JP15.4
- net DRILL_S1: no longer U3.2
- net DRILL_S2: no longer U3.12
- net ESTOP_LOCAL: no longer Q1.2, Q1.5, R13.1
- net GND: no longer C11.2, C12.2, JP10.1, JP11.1, JP15.1, JP6.1, LED10.C, LED11.C, LED8.C, LED9.C, Q1.3, Q1.6, Q6.1, Q6.4, Q7.1, Q7.4, U3.7, U4.7
- net LOWER_SWITCH: no longer JP11.2, R24.1
- net RC_S1: no longer JP6.3
- net RC_S2: no longer JP6.4
- net STEPPER_DIR: no longer JP7.2
- net STEPPER_EN: no longer JP7.3
- net STEPPER_STEP: no longer JP7.1
- net UPPER_SWITCH: no longer JP10.2, R23.1
Routing:
- net +3V3: track 162.1 -> 104.0 mm, vias 10 -> 8
- net RC_PWR: track 30.0 -> 0.00 mm
- net DRILL_EN: track 34.1 -> 9.44 mm, vias 2 -> 0
- net RELAY3_CNTRL: track 21.9 -> 0.00 mm, vias 2 -> 0
- net N$23: track 21.6 -> 0.00 mm, vias 2 -> 0
- net RELAY4_CNTRL: track 21.2 -> 0.00 mm
- net GND: track 111.5 -> 92.0 mm, vias 29 -> 20
- net N$25: track 15.2 -> 0.00 mm
- net RELAY2_CNTRL: track 14.8 -> 0.00 mm
- net RELAY1_CNTRL: track 14.8 -> 0.00 mm, vias 2 -> 0
- net N$22: track 13.1 -> 0.00 mm
- net ESTOP_RELAY: track 11.4 -> 0.00 mm
- net STEPPER_DIR: track 16.9 -> 7.48 mm
- net DRILL_RELAY_3: track 7.18 -> 0.00 mm
- net +12V: track 38.2 -> 31.2 mm
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
Commit message: PC2CAN ready for fab
Parts:
- removed JP12: M02LOCK, SparkFun-Connectors:1X02_LOCK
- removed Q5: INFINEON_2N7002_DW, npol-discrete:INFINEON_SOT363
- added C11: 10nF, rcl:C0603
- added C12: 0.1uF, rcl:C0603
- added JP6: (no value), SparkFun-Connectors:1X03_LOCK
- added JP7: USB-B, SparkFun-Connectors:USB-B-PTH
- added JP8: M02POLAR_LOCK, SparkFun-Connectors:MOLEX-1X2_LOCK
- added LED10, LED8, LED9: (no value), SparkFun-LED:LED-0603
- added Q1: INFINEON_2N7002_DW, npol-discrete:INFINEON_SOT363
- added R13, R23: 10k, rcl:R0603
- added R24: 620, rcl:R0603
- added U3: LTV-817, npol-digital:LITEON_DIL04_.3
- JP1: device SparkFun-Connectors:2X3 -> SparkFun-Connectors:1X05
- JP2: value M02LOCK -> (none); device SparkFun-Connectors:1X02_LOCK -> SparkFun-Connectors:2X3
- JP3: value ONSHORE_OST302-S141 -> M02LOCK; device npol-connectors:ONSHORE_OST302-S141 -> SparkFun-Connectors:1X02_LOCK
- JP4: value FTDI_DEVICE -> ONSHORE_OST302-S141; device SparkFun-Connectors:FTDI_DEVICE_SIDE -> npol-connectors:ONSHORE_OST302-S141
- JP5: value (none) -> FTDI_DEVICE; device SparkFun-Connectors:1X03_LOCK -> SparkFun-Connectors:FTDI_DEVICE_SIDE
- JP9: value M02POLAR_LOCK -> M02LOCK; device SparkFun-Connectors:MOLEX-1X2_LOCK -> SparkFun-Connectors:1X02_LOCK
- Q2: value INFINEON_2N7002_DW -> BS250F; device npol-discrete:INFINEON_SOT363 -> SparkFun-DiscreteSemi:SOT23-3
- Q4: value BS250F -> INFINEON_2N7002_DW; device SparkFun-DiscreteSemi:SOT23-3 -> npol-discrete:INFINEON_SOT363
- R15, R17: value 10k -> 470
- R18, R21: value 100k -> 10k
- R20, R22: value 10k -> 100k
- R25: value 620 -> 10k
- U2: value LTV-817 -> FT232RLSSOP; device npol-digital:LITEON_DIL04_.3 -> SparkFun-DigitalIC:SSOP28DB
- moved Q4 45.4 mm to (26.0, 50.8)
- moved JP5 44.7 mm to (55.2, 17.1), turned to 90 degrees
- moved JP4 42.6 mm to (5.08, 22.2), turned to 270 degrees
- moved JP1 37.2 mm to (49.5, 19.1), turned to 180 degrees
- moved JP3 31.7 mm to (33.7, 17.8)
- moved U2 29.9 mm to (51.4, 31.8), turned to 90 degrees
- moved JP2 28.9 mm to (14.0, 29.8), turned to 90 degrees
- moved R17 27.1 mm to (44.5, 31.8), turned to 180 degrees
- moved JP9 16.8 mm to (30.5, 51.4), turned to 270 degrees
- moved R26 16.8 mm to (26.0, 47.6), turned to 180 degrees
- moved R8 14.8 mm to (15.2, 41.9), flipped to the top
- moved R25 13.6 mm to (26.0, 45.1), turned to 180 degrees
- moved R14 13.6 mm to (33.0, 33.0), turned to 270 degrees
- moved LED4 9.86 mm to (11.4, 41.9), turned to 270 degrees
- moved H3 9.52 mm to (52.1, 49.5)
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Connections:
- removed net DRILL_EN: U1.59
- removed net DRILL_ISENSE_/FAULT: U1.24
- removed net DRILL_ISENSE_FAULT_EN: U1.77
- removed net DRILL_ISENSE_VIOUT: U1.79
- removed net DRILL_ISENSE_VZCR: U1.78
- removed net DRILL_S1: U1.58
- removed net DRILL_S2: U1.57
- removed net LOWER_SWITCH: U1.29
- removed net RC_RXD: R14.2, SJ3.3, SJ4.1, U1.52
- removed net RC_S1: SJ3.2
- removed net RC_S2: SJ4.2
- removed net RC_TXD: R15.2, SJ3.1, SJ4.3, U1.51
- removed net STEPPER_DIR: U1.6
- removed net STEPPER_EN: U1.7
- removed net STEPPER_STEP: U1.23
- removed net UPPER_SWITCH: U1.30
- new net N$14: JP7.D+, U2.15
- new net N$15: JP7.D-, U2.16
- new net N$16: LED8.C, R15.2
- new net N$17: LED9.C, R17.2
- new net N$18: R15.1, U2.23
- new net N$19: R17.1, U2.22
- new net N$20: C12.1, U2.17
- new net N$21: Q4.3, R26.2
- new net N$22: LED10.C, R26.1
- new net NU_P3.7: JP1.5, U1.44
- new net NU_P4.0: JP1.4, U1.45
- new net NU_P4.1: JP1.3, U1.46
- new net NU_P4.2: JP1.2, U1.47
- new net NU_P4.3: JP1.1, U1.48
- new net USB_RX: SJ3.2, U2.1
- new net USB_RXD: R13.2, SJ3.3, SJ4.1, U1.52
- new net USB_TX: SJ4.2, U2.5
- new net USB_TXD: R14.2, SJ3.1, SJ4.3, U1.51
- new net VBUS: C11.1, JP7.VBUS, LED8.A, LED9.A, U2.20, U2.4
- net +12V: now also Q3.2, R21.2; no longer Q4.2, R20.2
- net +3V3: now also JP3.1, JP6.2, LED10.A, R25.1; no longer JP2.1, JP5.2, R26.1
- net +5V: now also Q2.2, R18.2; no longer Q3.2, R17.2
- net 12VSENSE: now also R22.1, R23.2; no longer R21.1, R22.2
- net 5VSENSE: now also R19.1, R20.2; no longer R18.1, R19.2
- net ESTOP+: now also JP8.1, R24.2; no longer JP9.1, R25.2
- net ESTOP-: now also JP8.2, U3.2; no longer JP9.2, U2.2
- net ESTOP_LOCAL: now also JP9.1, Q4.5, Q4.6, R25.2; no longer JP12.1, Q5.6, R26.2
- net ESTOP_LOCAL_INV: now also Q4.2, U3.4; no longer Q5.2, U2.4
- net GND: now also C11.2, C12.2, JP2.2, JP4.9, JP5.P$6, JP7.GND, JP9.2, Q1.1, Q1.4, Q4.1, Q4.4, R13.1, R20.1, R23.1, U2.18, U2.21, U2.25, U2.26, U2.7, U3.3; no longer JP1.2, JP12.2, JP3.9, JP4.P$6, Q2.1, Q2.4, Q5.1, R15.1, R19.1, R22.1, U2.3
- net N$1: now also JP3.2, JP5.P$4; no longer JP2.2, JP4.P$4
- net N$10: now also Q1.6, Q2.1, R18.1; no longer Q2.6, Q3.1, R17.1
- net N$11: now also Q3.3, R22.2; no longer Q4.3, R21.2
- net N$12: now also Q1.2, Q1.5; no longer Q2.2, Q2.5
- net N$13: now also R24.1, U3.1; no longer R25.1, U2.1
- net N$9: now also Q2.3, R19.2; no longer Q3.3, R18.2
- net NU_P6.3: now also JP2.5; no longer JP1.5
- net NU_P6.4: now also JP2.6; no longer JP1.6
- net NU_P6.5: now also JP2.3; no longer JP1.3
- net NU_P6.6: now also JP2.4; no longer JP1.4
- net NU_P6.7: now also JP2.1; no longer JP1.1
- net RXI: now also JP5.P$3; no longer JP4.P$3
- net SBWTCK: now also JP4.7; no longer JP3.7
- net SBWTDIO: now also JP4.1; no longer JP3.1
- net TXO: now also JP5.P$2; no longer JP4.P$2
- net VCC_TARGET: now also JP4.4, JP6.1; no longer JP3.4, JP5.1
- net VCC_TOOL: now also JP4.2, JP6.3; no longer JP3.2, JP5.3
- net VTAP_EN: now also Q1.3, Q3.1, R21.1; no longer Q2.3, Q4.1, R20.1
Routing:
- net DRILL_ISENSE_/FAULT: track 74.6 -> 0.00 mm, vias 2 -> 0
- net +5V: track 69.3 -> 10.6 mm
- net ESTOP_LOCAL: track 134.1 -> 75.9 mm, vias 4 -> 2
- net STEPPER_STEP: track 43.9 -> 0.00 mm
- net DRILL_ISENSE_FAULT_EN: track 40.4 -> 0.00 mm
- net DRILL_ISENSE_VZCR: track 36.7 -> 0.00 mm
- net DRILL_ISENSE_VIOUT: track 35.7 -> 0.00 mm
- net USB_TX: track 0.00 -> 32.0 mm, vias 0 -> 2
- net LOWER_SWITCH: track 28.5 -> 0.00 mm, vias 1 -> 0
- net VBUS: track 0.00 -> 27.4 mm
- net SBWTCK: track 19.6 -> 46.6 mm, vias 0 -> 2
- net UPPER_SWITCH: track 24.7 -> 0.00 mm, vias 1 -> 0
- net USB_RX: track 0.00 -> 20.8 mm
- net NU_P4.3: track 0.00 -> 20.4 mm
- net USB_RXD: track 0.00 -> 18.3 mm, vias 0 -> 2
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Other:
- board size 57.1 x 63.5 mm -> 57.1 x 54.6 mm
- board text added: "CLEANUP Team NSH PC-CAN Controller"
- board text added: "ESTOP TEST"
- board text added: "P3.7"
- board text added: "P4.0"
- board text added: "P4.1"
- board text added: "P4.2"
- board text added: "P4.3"
- board text added: "RX"
- board text added: "TX"
- board text removed: "CLEANUP Team NSH Mobility-Elim Controller"
- board text removed: "PWR"
- board text removed: "RLY1"
- board text removed: "RLY2"
- board text removed: "RLY3"
- board text removed: "RLY4"
- board text removed: "S1"
- board text removed: "S2"

Commit message: Power Controller, Elim-Mobility Controller, and PC2CAN sent to FAB
Parts:
- added JP10: (no value), SparkFun-Connectors:1X03_LOCK
- added R27: 10k, rcl:R0603
- added R28: 10M, rcl:R0603
Connections:
- net +3V3: now also R27.1
- net ESTOP_LOCAL_INV: now also R27.2, R28.1
- net GND: now also JP10.1, R28.2
- net USB_RX: now also JP10.3
- net USB_TX: now also JP10.2
Routing:
- net +3V3: track 95.0 -> 110.2 mm
- net USB_RX: track 20.8 -> 34.8 mm
- net USB_TX: track 32.0 -> 41.0 mm
- net ESTOP_LOCAL_INV: track 8.62 -> 16.1 mm
Other:
- board text added: "RXD"
- board text added: "TXD"
Changed lines of the file:
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@@
 <text x="34.29" y="48.26" size="0.8128" layer="25" rot="R90">ESTOP
 TEST</text>
+<text x="50.165" y="41.275" size="0.8128" layer="25" rot="R90">GND</text>
+<text x="52.705" y="41.275" size="0.8128" layer="25" rot="R90">TXD</text>
+<text x="55.245" y="41.275" size="0.8128" layer="25" rot="R90">RXD</text>
 </plain>
 <attributes>
@@
 <element name="JP7" library="SparkFun-Connectors" package="USB-B-PTH" value="USB-B" x="40.64" y="41.91" smashed="yes" rot="R270">
 <attribute name="PROD_ID" value="CONN-08278" x="12.065" y="41.91" size="1.778" layer="27" rot="R270" display="off"/>
-<attribute name="NAME" x="47.625" y="41.275" size="0.8128" layer="25" rot="R270"/>
+<attribute name="NAME" x="34.29" y="37.465" size="0.8128" layer="25"/>
 </element>
 <element name="C11" library="rcl" package="C0603" value="10nF" x="38.735" y="36.83" smashed="yes" rot="R180">
@@
 </element>
 <element name="Q4" library="npol-discrete" package="INFINEON_SOT363" value="INFINEON_2N7002_DW" x="26.035" y="50.8" smashed="yes" rot="R270">
-<attribute name="NAME" x="26.035" y="52.705" size="0.8128" layer="25"/>
+<attribute name="NAME" x="23.495" y="52.705" size="0.8128" layer="25"/>
 </element>
 <element name="LED10" library="SparkFun-LED" package="LED-0603" value="" x="28.575" y="46.355" smashed="yes">
@@
 <element name="R26" library="rcl" package="R0603" value="10k" x="26.035" y="47.625" smashed="yes" rot="R180">
 <attribute name="NAME" x="23.495" y="48.895" size="0.8128" layer="25" rot="R270"/>
+</element>
+<element name="R27" library="rcl" package="R0603" value="10k" x="26.67" y="53.34" smashed="yes" rot="R180">
+<attribute name="NAME" x="28.575" y="53.34" size="0.8128" layer="25"/>
+</element>
+<element name="R28" library="rcl" package="R0603" value="10M" x="21.59" y="48.26" smashed="yes" rot="MR90">
+<attribute name="NAME" x="22.86" y="47.625" size="0.8128" layer="26" rot="MR90"/>
+</element>
+<element name="JP10" library="SparkFun-Connectors" package="1X03_LOCK" value="" x="49.53" y="39.37" smashed="yes">
+<attribute name="NAME" x="47.7012" y="38.0238" size="0.8128" layer="25" ratio="10" rot="R90"/>
+<attribute name="VALUE" x="48.26" y="36.195" size="1.27" layer="27"/>
 </element>
 </elements>
@@
 <wire x1="25.235" y1="51.45" x2="24.75" y2="51.45" width="0.3048" layer="1"/>
 <wire x1="24.75" y1="51.45" x2="24.13" y2="52.07" width="0.3048" layer="1"/>
+<contactref element="R28" pad="2"/>
+<contactref element="JP10" pad="1"/>
 </signal>
 <signal name="CAN_STBY">
@@
 <wire x1="26.885" y1="45.085" x2="28.055" y2="45.085" width="0.3048" layer="1"/>
 <wire x1="28.055" y1="45.085" x2="28.575" y2="45.605" width="0.3048" layer="1"/>
+<contactref element="R27" pad="1"/>
+<wire x1="27.52" y1="53.34" x2="31.75" y2="53.34" width="0.3048" layer="1"/>
+<wire x1="31.75" y1="53.34" x2="32.385" y2="52.705" width="0.3048" layer="1"/>
+<wire x1="32.385" y1="52.705" x2="32.385" y2="46.99" width="0.3048" layer="1"/>
+<wire x1="32.385" y1="46.99" x2="31.115" y2="45.72" width="0.3048" layer="1"/>
+<wire x1="31.115" y1="45.72" x2="28.69" y2="45.72" width="0.3048" layer="1"/>
+<wire x1="28.69" y1="45.72" x2="28.575" y2="45.605" width="0.3048" layer="1"/>
 </signal>
 <signal name="SBWTDIO">
@@
 <wire x1="22.86" y1="50.8" x2="21.59" y2="49.53" width="0.3048" layer="1"/>
 <wire x1="21.59" y1="49.53" x2="21.59" y2="45.085" width="0.3048" layer="1"/>
+<contactref element="R27" pad="2"/>
+<contactref element="R28" pad="1"/>
+<wire x1="21.59" y1="47.41" x2="21.59" y2="45.085" width="0.3048" layer="16"/>
+<wire x1="25.82" y1="53.34" x2="23.495" y2="53.34" width="0.3048" layer="1"/>
+<wire x1="23.495" y1="53.34" x2="22.86" y2="52.705" width="0.3048" layer="1"/>
+<wire x1="22.86" y1="52.705" x2="22.86" y2="50.8" width="0.3048" layer="1"/>
 </signal>
 <signal name="N$13">
@@
 <wire x1="53.975" y1="27.305" x2="54.871" y2="27.305" width="0.254" layer="1"/>
 <wire x1="54.871" y1="27.305" x2="55.091" y2="27.525" width="0.254" layer="1"/>
+<contactref element="JP10" pad="3"/>
+<wire x1="55.091" y1="27.525" x2="56.1" y2="27.525" width="0.3048" layer="1"/>
+<wire x1="56.1" y1="27.525" x2="56.515" y2="27.94" width="0.3048" layer="1"/>
+<wire x1="56.515" y1="27.94" x2="56.515" y2="37.592" width="0.3048" layer="1"/>
+<wire x1="56.515" y1="37.592" x2="54.61" y2="39.497" width="0.3048" layer="1"/>
 </signal>
 <signal name="USB_TX">
@@
 <wire x1="55.091" y1="30.125" x2="53.06" y2="30.125" width="0.254" layer="1"/>
 <wire x1="53.06" y1="30.125" x2="52.705" y2="30.48" width="0.254" layer="1"/>
+<contactref element="JP10" pad="2"/>
+<wire x1="52.705" y1="30.48" x2="52.07" y2="31.115" width="0.3048" layer="1"/>
+<wire x1="52.07" y1="31.115" x2="52.07" y2="39.243" width="0.3048" layer="1"/>
 </signal>
 <signal name="N$20">
