File: SensorController/SensorController.brd (EAGLE design)
At the start: 57.1 x 54.6 mm, 76 parts, among them J11 M10X2, Q1 INFINEON_2N7002_DW, Q2 BS250F, Q3 BS250F, Q4 INFINEON_2N7002_DW, Q5 INFINEON_2N7002_DW, U1 MSP430F5521/5/7/9_PN80

Commit message: Deleted irrelevant parts from SensorController
Parts:
- removed LED10, LED8, LED9: (no value), SparkFun-LED:LED-0603
- removed Q4, Q5: INFINEON_2N7002_DW, npol-discrete:INFINEON_SOT363
- removed R13, R14, R22, R23: 10k, rcl:R0603
- removed R24, R26: 470, rcl:R0603
- removed R25, R27: 330, rcl:R0603
- removed R28: 10M, rcl:R0603
- removed SJ3, SJ4: (no value), microbuilder:SOLDERJUMPER_2WAY_OPEN_0603
- removed XB1: XBEE, microbuilder:XBEE
- added JP10, JP8, JP9: (no value), SparkFun-Connectors:1X04
- JP7: value M02POLAR_LOCK -> (none); device SparkFun-Connectors:MOLEX-1X2_LOCK -> SparkFun-Connectors:1X04
- moved JP7 33.9 mm to (47.6, 40.6), turned to 0 degrees
Connections:
- removed net ESTOP_INV: LED8.C, Q4.5, Q4.6, R23.2, R28.1, U1.22
- removed net ESTOP_OUT: JP7.1, Q4.2, Q5.6, R25.2
- removed net ESTOP_PULLDOWN: Q5.2, Q5.5, R22.1, U1.23
- removed net N$17: LED9.C, R26.1
- removed net XBEE_DIN: SJ3.2, XB1.3
- removed net XBEE_DOUT: SJ4.2, XB1.2
- removed net XBEE_RXD: R13.2, SJ3.3, SJ4.1, U1.52
- removed net XBEE_TXD: R14.2, SJ3.1, SJ4.3, U1.51
- net +12V: now also JP10.1, JP7.1, JP8.1, JP9.1; no longer R25.1
- net +3V3: now also JP10.2, JP7.2, JP8.2, JP9.2; no longer LED10.A, LED9.A, R23.1, R24.1, XB1.1
- net GND: now also JP10.3, JP7.3, JP8.3, JP9.3; no longer JP7.2, Q4.1, Q4.4, Q5.1, Q5.4, R13.1, R14.1, R22.2, R28.2, XB1.10
- net N$13: now also JP10.4; no longer Q5.3, R27.2
- net N$14: now also JP9.4; no longer LED10.C, R27.1
- net N$15: now also JP8.4; no longer LED8.A, R24.2
- net N$16: now also JP7.4; no longer Q4.3, R26.2
Routing:
- net ESTOP_INV: track 74.0 -> 0.00 mm, vias 2 -> 0
- net ESTOP_PULLDOWN: track 58.1 -> 0.00 mm, vias 2 -> 0
- net ESTOP_OUT: track 29.5 -> 0.00 mm
- net XBEE_DIN: track 28.6 -> 0.00 mm
- net XBEE_RXD: track 24.5 -> 0.00 mm, vias 2 -> 0
- net XBEE_DOUT: track 18.5 -> 0.00 mm, vias 1 -> 0
- net XBEE_TXD: track 16.5 -> 0.00 mm, vias 2 -> 0
- net GND: track 97.8 -> 84.1 mm, vias 25 -> 18
- net N$17: track 10.9 -> 0.00 mm
- net +3V3: track 111.6 -> 101.0 mm
- net N$14: track 3.82 -> 0.00 mm
- net N$15: track 2.57 -> 0.00 mm
- net N$13: track 2.36 -> 0.00 mm
- net N$16: track 2.17 -> 0.00 mm
- net +12V: track 91.7 -> 91.1 mm
- removed copper zone on layer 1, net +3V3
