File: SensorController/SensorController.sch (EAGLE design)
At the start: 76 parts, among them J11 M10X2, Q1 INFINEON_2N7002_DW, Q2 BS250F, Q3 BS250F, Q4 INFINEON_2N7002_DW, Q5 INFINEON_2N7002_DW, U1 MSP430F5521/5/7/9_PN80

Commit message: Deleted irrelevant parts from SensorController
Parts:
- removed LED10, LED8, LED9: (no value), SparkFun-LED:LED0603
- removed Q4, Q5: INFINEON_2N7002_DW, npol-discrete:INFINEON_2N7002_DW
- removed R13, R14, R22, R23: 10k, rcl:R-US_R0603
- removed R24, R26: 470, rcl:R-US_R0603
- removed R25, R27: 330, rcl:R-US_R0603
- removed R28: 10M, rcl:R-US_R0603
- removed SJ3, SJ4: (no value), microbuilder:SOLDERJUMPER_2WAY0603
- removed XB1: XBEE, microbuilder:XBEE
- added JP10, JP8, JP9: (no value), SparkFun-Connectors:M04PTH
- JP7: value M02POLAR_LOCK -> (none); device SparkFun-Connectors:M02POLAR_LOCK -> SparkFun-Connectors:M04PTH
Connections:
- removed net ESTOP_INV: LED8.C, Q4G$1.DRAIN, Q4G$2.GATE, R23.2, R28.1, U1.P1.1/TA0.0
- removed net ESTOP_OUT: JP7.1, Q4G$1.GATE, Q5G$1.DRAIN, R25.2
- removed net ESTOP_PULLDOWN: Q5G$1.GATE, Q5G$2.GATE, R22.1, U1.P1.2/TA0.1
- removed net N$17: LED9.C, R26.1
- removed net XBEE_DIN: SJ3.2, XB1.DIN/!CONFIG
- removed net XBEE_DOUT: SJ4.2, XB1.DOUT
- removed net XBEE_RXD: R13.2, SJ3.3, SJ4.1, U1.P4.5/PM_UCA1RXD/PM_UCA1SOMI
- removed net XBEE_TXD: R14.2, SJ3.1, SJ4.3, U1.P4.4/PM_UCA1TXD/PM_UCA1SIMO
- net +12V: now also JP10.1, JP7.1, JP8.1, JP9.1; no longer R25.1
- net +3V3: now also JP10.2, JP7.2, JP8.2, JP9.2; no longer LED10.A, LED9.A, R23.1, R24.1, XB1.VCC
- net GND: now also JP10.3, JP7.3, JP8.3, JP9.3; no longer JP7.2, Q4G$1.SOURCE, Q4G$2.SOURCE, Q5G$1.SOURCE, Q5G$2.SOURCE, R13.1, R14.1, R22.2, R28.2, XB1.GND
- net N$13: now also JP10.4; no longer Q5G$2.DRAIN, R27.2
- net N$14: now also JP9.4; no longer LED10.C, R27.1
- net N$15: now also JP8.4; no longer LED8.A, R24.2
- net N$16: now also JP7.4; no longer Q4G$2.DRAIN, R26.2
Other:
- note removed: "Active low output"
- note removed: "ESTOP"
